File: efr32bg_breakout.kicad_sch (KiCad schematic)
At the start: 12 parts, among them J1 Conn_01x06, J2 Conn_01x10, J3 Conn_01x10, SW1 SW_Push, U1 E104-BT53A3

Commit message: use 0603 leds
Parts:
- D1, D2: footprint LED_SMD:LED_0402_1005Metric -> LED_SMD:LED_0603_1608Metric
Changed lines of the file:
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@@
 			)
 		)
-		(property "Footprint" "LED_SMD:LED_0402_1005Metric"
+		(property "Footprint" "LED_SMD:LED_0603_1608Metric"
 			(at 81.28 45.72 0)
 			(effects
@@
 			)
 		)
-		(property "Footprint" "LED_SMD:LED_0402_1005Metric"
+		(property "Footprint" "LED_SMD:LED_0603_1608Metric"
 			(at 252.73 113.03 0)
 			(effects
